Commit message: rm gripper convex hull geometries, small boxes for wrist force-torque sensors.

File: deps/Atlas/atlas.urdf (robot description, URDF)
Before this commit: robot atlas, 70 links, 69 joints
Links:
- link l_hand_force_torque: geometry 
- link left_palm: geometry 
- link r_hand_force_torque: geometry 
- link right_palm: geometry 
